File: kicad/IP5306_Module.kicad_pcb (KiCad board)
At the start: 2 copper layers, 50 x 20 mm, 26 parts, among them J1 USB_C_Receptacle_USB2.0_16P, J2 USB_A, J3 Conn_01x02, SW1 SW_Push, U1 IP5306

Commit message: changes
Parts:
- added G***: LOGO, customimages:linuxpenguin, B.Cu at (49.4, 40.0)
